File: kicad/kicad.kicad_sch (KiCad schematic)
At the start: 53 parts, among them U1 TL071, U10 TL071, U11 NE555P, U2 TL071, U3 TL071, U4 TL071, U5 TL071, U6 TL071, U7 TL071, U8 TL071, U9 TL071

Commit message: Update kicad project
Parts:
- added C13, C15: C, symbol Device:C
- added D1, D2: 1N4007, Diode_THT:D_DO-41_SOD81_P10.16mm_Horizontal, symbol Diode:1N4007
- added J1, J10, J11, J12, J2, J3, J4, J5, J6, J7, J8, J9: Conn_01x06_Pin, symbol Connector:Conn_01x06_Pin
- added R30, R31, R32: R, symbol Device:R
- added RV1, RV2: R_Potentiometer, symbol Device:R_Potentiometer
- added U12: TL071, symbol Amplifier_Operational:TL071
Connections:
- net GND: now also J1.3 (Pin_3), J10.3 (Pin_3), J11.3 (Pin_3), J12.3 (Pin_3), J2.3 (Pin_3), J3.3 (Pin_3), J4.3 (Pin_3), J5.3 (Pin_3), J6.3 (Pin_3), J7.3 (Pin_3), J8.3 (Pin_3), J9.3 (Pin_3), R31.2
- net module 1 +VCC: now also J1.1 (Pin_1); no longer U10.7 (V+), U3.7 (V+), U4.7 (V+), U5.7 (V+), U6.7 (V+), U7.7 (V+), U8.7 (V+), U9.7 (V+)
- net module 1 -VCC: now also J1.2 (Pin_2); no longer U10.4 (V-), U3.4 (V-), U4.4 (V-), U5.4 (V-), U6.4 (V-), U7.4 (V-), U8.4 (V-), U9.4 (V-)
- net module 1 In1: now also J1.4 (Pin_4), J1.5 (Pin_5); no longer C2.2, C8.2, C9.2, R12.1, R17.1, R25.1, R6.1, R8.2, R9.2
- net module 1 Out: now also J1.6 (Pin_6); no longer C1.1, C4.1, C7.2, R10.2, R11.1, R14.1, R19.1, R20.2, R23.1, R24.2, R27.2, R29.1, R7.1, U10.6, U3.6, U4.6, U5.6, U6.6, U7.6, U8.6, U9.6
- net module 2 +VCC: now also J2.1 (Pin_1)
- net module 2 -VCC: now also J2.2 (Pin_2)
- net module 2 In1: now also J2.4 (Pin_4)
- net module 2 In2: now also J2.5 (Pin_5)
- net module 2 Out: now also J2.6 (Pin_6)
- net module 11 -VCC: now reaches U11.1 (GND)
- net module 11 -VCC: now also C13.2, C15.1, J11.2 (Pin_2)
- net at U11.2 (TR): now also U11.6 (THR), C13.1, RV2.2
- net module 11 Out: now reaches U11.3 (Q)
- net module 11 Out: now also J11.6 (Pin_6)
- net module 11 +VCC: now reaches U11.4 (R)
- net module 11 +VCC: now also U11.8 (VCC), J11.1 (Pin_1), R30.1
- net at U11.5 (CV): now also C15.2
- net at U11.7 (DIS): now also D1.2 (A), D2.1 (K), RV1.1
- new net: D2.2 (A), RV2.1
- new net: D1.1 (K), RV2.3
- new net: R31.1, R32.2, U12.2 (-)
- new net: R30.2, RV1.2, RV1.3
- new net module 10 +VCC: J10.1 (Pin_1), U10.7 (V+)
- new net module 10 -VCC: J10.2 (Pin_2), U10.4 (V-)
- new net module 10 In1: C9.2, J10.4 (Pin_4), J10.5 (Pin_5), R25.1
- new net module 10 Out: J10.6 (Pin_6), R27.2, R29.1, U10.6
- new net module 11 In1: J11.4 (Pin_4)
- new net module 11 In2: J11.5 (Pin_5)
- new net module 12 +VCC: J12.1 (Pin_1), U12.7 (V+)
- new net module 12 -VCC: J12.2 (Pin_2), U12.4 (V-)
- new net module 12 In1: J12.4 (Pin_4), J12.5 (Pin_5), U12.3 (+)
- new net module 12 Out: J12.6 (Pin_6), R32.1, U12.6
- new net module 3 +VCC: J3.1 (Pin_1), U5.7 (V+)
- new net module 3 -VCC: J3.2 (Pin_2), U5.4 (V-)
- new net module 3 In1: C2.2, J3.4 (Pin_4), J3.5 (Pin_5)
- new net module 3 Out: J3.6 (Pin_6), R10.2, U5.6
- new net module 4 +VCC: J4.1 (Pin_1), U4.7 (V+)
- new net module 4 -VCC: J4.2 (Pin_2), U4.4 (V-)
- new net module 4 In1: J4.4 (Pin_4), J4.5 (Pin_5), R9.2
- new net module 4 Out: C1.1, J4.6 (Pin_6), U4.6
- new net module 5 +VCC: J5.1 (Pin_1), U6.7 (V+)
- new net module 5 -VCC: J5.2 (Pin_2), U6.4 (V-)
- new net module 5 In1: J5.4 (Pin_4), J5.5 (Pin_5), R8.2
- new net module 5 Out: C4.1, J5.6 (Pin_6), R11.1, U6.6
- new net module 6 +VCC: J6.1 (Pin_1), U7.7 (V+)
- new net module 6 -VCC: J6.2 (Pin_2), U7.4 (V-)
- new net module 6 In1: J6.4 (Pin_4), J6.5 (Pin_5), R12.1
- new net module 6 Out: C7.2, J6.6 (Pin_6), R14.1, U7.6
- new net module 7 +VCC: J7.1 (Pin_1), U9.7 (V+)
- new net module 7 -VCC: J7.2 (Pin_2), U9.4 (V-)
- new net module 7 In1: J7.4 (Pin_4), J7.5 (Pin_5), R17.1
- new net module 7 Out: J7.6 (Pin_6), R23.1, R24.2, U9.6
- new net module 8 +VCC: J8.1 (Pin_1), U3.7 (V+)
- new net module 8 -VCC: J8.2 (Pin_2), U3.4 (V-)
- new net module 8 In1: J8.4 (Pin_4), J8.5 (Pin_5), R6.1
- new net module 8 Out: J8.6 (Pin_6), R7.1, U3.6
- new net module 9 +VCC: J9.1 (Pin_1), U8.7 (V+)
- new net module 9 -VCC: J9.2 (Pin_2), U8.4 (V-)
- new net module 9 In1: C8.2, J9.4 (Pin_4), J9.5 (Pin_5)
- new net module 9 Out: J9.6 (Pin_6), R19.1, R20.2, U8.6
- no-connect marks 0 -> 22
Other:
- note added: "Circuito NE555 gerador PWM"
- note added: "Circuito Não Inversor"
- moved on the sheet: C1, C10, C11, C12, C14, C2, C5, C6, C7, C8, C9, R10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
