File: modules/NE555PWMGenerator/NE555PWMGenerator.kicad_sch (KiCad schematic)
At the start: 9 parts

Commit message: Little changes on each schematic
Changed lines of the file:
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@@
   (junction (at 97.79 104.14) (diameter 0) (color 0 0 0 0)
   )
-  (junction (at 119.38 130.81) (diameter 0) (color 0 0 0 0)
-  )
   (junction (at 101.6 144.78) (diameter 0) (color 0 0 0 0)
   )
   (junction (at 102.87 109.22) (diameter 0) (color 0 0 0 0)
-  )
-  (junction (at 119.38 110.49) (diameter 0) (color 0 0 0 0)
   )
   (junction (at 96.52 129.54) (diameter 0) (color 0 0 0 0)
@@
     )
   )
-  (symbol (lib_id "power:PWR_FLAG") (at 119.38 110.49 90) (unit 1)
-    (in_bom yes) (on_board yes) (dnp no) (fields_autoplaced)
-    (property "Reference" "#FLG?" (at 117.475 110.49 0)
-      (effects (font (size 1.27 1.27)) hide)
-    )
-    (property "Value" "PWR_FLAG" (at 114.3 110.49 0)
-      (effects (font (size 1.27 1.27)) hide)
-    )
-    (property "Footprint" "" (at 119.38 110.49 0)
-      (effects (font (size 1.27 1.27)) hide)
-    )
-    (property "Datasheet" "~" (at 119.38 110.49 0)
-      (effects (font (size 1.27 1.27)) hide)
-    )
-    (pin "1")
-    (instances
-      (project "kicad"
-        (path "/1ce81232-195d-4047-8575-458c62622b55"
-          (reference "#FLG?") (unit 1)
-        )
-      )
-      (project "NE555PWMGenerator"
-        (path "/28625a42-f066-4c35-899c-06e6b47fd65b"
-          (reference "#FLG023") (unit 1)
-        )
-      )
-    )
-  )
   (symbol (lib_id "Connector:Conn_01x06_Pin") (at 163.83 137.16 0) (mirror y) (unit 1)
     (in_bom yes) (on_board yes) (dnp no)
@@
         )
       )
-    )
-  )
-  (symbol (lib_id "power:PWR_FLAG") (at 119.38 130.81 90) (unit 1)
-    (in_bom yes) (on_board yes) (dnp no) (fields_autoplaced)
-    (property "Reference" "#FLG?" (at 117.475 130.81 0)
-      (effects (font (size 1.27 1.27)) hide)
-    )
-    (property "Value" "PWR_FLAG" (at 114.3 130.81 0)
-      (effects (font (size 1.27 1.27)) hide)
-    )
-    (property "Footprint" "" (at 119.38 130.81 0)
-      (effects (font (size 1.27 1.27)) hide)
-    )
-    (property "Datasheet" "~" (at 119.38 130.81 0)
-      (effects (font (size 1.27 1.27)) hide)
-    )
-    (pin "1")
-    (instances
-      (project "kicad"
-        (path "/1ce81232-195d-4047-8575-458c62622b55"
-          (reference "#FLG?") (unit 1)
-        )
-      )
-      (project "NE555PWMGenerator"
-        (path "/28625a42-f066-4c35-899c-06e6b47fd65b"
-          (reference "#FLG025") (unit 1)
-        )
-      )
