File: modules/bandPassSecondOrderSK/bandPassSecondOrderSK.kicad_sch (KiCad schematic)
At the start: 9 parts

Commit message: Update moudules
Parts:
- removed R?: R, Resistor_THT:R_Axial_DIN0207_L6.3mm_D2.5mm_P7.62mm_Horizontal, symbol Device:R
- added R?: R, Resistor_THT:R_Axial_DIN0207_L6.3mm_D2.5mm_P7.62mm_Horizontal, symbol Device:R
Connections:
- net GND: now also R?.1
- net at U?.2 (-): now also R?.2, R?.2
Changed lines of the file:
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@@
   (junction (at 176.53 59.69) (diameter 0) (color 0 0 0 0)
+  )
+  (junction (at 209.55 64.77) (diameter 0) (color 0 0 0 0)
   )
   (junction (at 165.1 48.26) (diameter 0) (color 0 0 0 0)
@@
     (stroke (width 0) (type default))
   )
-  (wire (pts (xy 194.31 64.77) (xy 180.34 64.77))
-    (stroke (width 0) (type default))
-  )
   (wire (pts (xy 180.34 64.77) (xy 180.34 54.61))
     (stroke (width 0) (type default))
@@
     (stroke (width 0) (type default))
   )
-  (wire (pts (xy 201.93 64.77) (xy 209.55 64.77))
+  (wire (pts (xy 180.34 64.77) (xy 209.55 64.77))
     (stroke (width 0) (type default))
   )
@@
         (path "/2121d978-39fd-4952-bc51-dbaf52d83413"
           (reference "#PWR01") (unit 1)
+        )
+      )
+    )
+  )
+  (symbol (lib_id "Device:R") (at 209.55 68.58 0) (mirror x) (unit 1)
+    (in_bom yes) (on_board yes) (dnp no)
+    (property "Reference" "R?" (at 213.36 69.85 90)
+      (effects (font (size 1.27 1.27)) (justify left))
+    )
+    (property "Value" "R" (at 213.36 67.31 90)
+      (effects (font (size 1.27 1.27)) (justify left) hide)
+    )
+    (property "Footprint" "Resistor_THT:R_Axial_DIN0207_L6.3mm_D2.5mm_P7.62mm_Horizontal" (at 207.772 68.58 90)
+      (effects (font (size 1.27 1.27)) hide)
+    )
+    (property "Datasheet" "~" (at 209.55 68.58 0)
+      (effects (font (size 1.27 1.27)) hide)
+    )
+    (pin "1")
+    (pin "2")
+    (instances
+      (project "kicad"
+        (path "/1ce81232-195d-4047-8575-458c62622b55"
+          (reference "R?") (unit 1)
+        )
+      )
+      (project "bandPassSecondOrderSK"
+        (path "/2121d978-39fd-4952-bc51-dbaf52d83413"
+          (reference "R4") (unit 1)
         )
       )
@@
     )
   )
-  (symbol (lib_id "Device:R") (at 198.12 64.77 90) (mirror x) (unit 1)
-    (in_bom yes) (on_board yes) (dnp no)
-    (property "Reference" "R?" (at 196.85 68.58 90)
-      (effects (font (size 1.27 1.27)) (justify left))
-    )
-    (property "Value" "R" (at 199.39 68.58 90)
-      (effects (font (size 1.27 1.27)) (justify left) hide)
-    )
-    (property "Footprint" "Resistor_THT:R_Axial_DIN0207_L6.3mm_D2.5mm_P7.62mm_Horizontal" (at 198.12 62.992 90)
-      (effects (font (size 1.27 1.27)) hide)
-    )
-    (property "Datasheet" "~" (at 198.12 64.77 0)
-      (effects (font (size 1.27 1.27)) hide)
-    )
-    (pin "1")
-    (pin "2")
-    (instances
-      (project "kicad"
-        (path "/1ce81232-195d-4047-8575-458c62622b55"
-          (reference "R?") (unit 1)
-        )
-      )
-      (project "bandPassSecondOrderSK"
-        (path "/2121d978-39fd-4952-bc51-dbaf52d83413"
-          (reference "R4") (unit 1)
-        )
-      )
+  (symbol (lib_id "power:GND") (at 209.55 72.39 0) (unit 1)
+    (in_bom yes) (on_board yes) (dnp no)
+    (property "Reference" "#PWR?" (at 209.55 78.74 0)
+      (effects (font (size 1.27 1.27)) hide)
+    )
+    (property "Value" "GND" (at 209.55 76.2 0)
+      (effects (font (size 1.27 1.27)) hide)
+    )
+    (property "Footprint" "" (at 209.55 72.39 0)
+      (effects (font (size 1.27 1.27)) hide)
+    )
+    (property "Datasheet" "" (at 209.55 72.39 0)
+      (effects (font (size 1.27 1.27)) hide)
+    )
+    (pin "1")
+    (instances
+      (project "kicad"
+        (path "/1ce81232-195d-4047-8575-458c62622b55"
+          (reference "#PWR?") (unit 1)
+        )
+      )
+      (project "bandPassSecondOrderSK"
+        (path "/2121d978-39fd-4952-bc51-dbaf52d83413"
+          (reference "#PWR04") (unit 1)
+        )
+      )

Commit message: Little changes on each schematic
Other:
- moved on the sheet: R?
Changed lines of the file:
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@@
   (junction (at 176.53 59.69) (diameter 0) (color 0 0 0 0)
   )
-  (junction (at 209.55 64.77) (diameter 0) (color 0 0 0 0)
+  (junction (at 209.55 66.04) (diameter 0) (color 0 0 0 0)
   )
   (junction (at 165.1 48.26) (diameter 0) (color 0 0 0 0)
-  )
-  (junction (at 185.42 59.69) (diameter 0) (color 0 0 0 0)
   )
   (junction (at 209.55 52.07) (diameter 0) (color 0 0 0 0)
@@
     (stroke (width 0) (type default))
   )
-  (wire (pts (xy 209.55 64.77) (xy 209.55 60.96))
+  (wire (pts (xy 209.55 60.96) (xy 209.55 66.04))
     (stroke (width 0) (type default))
   )
@@
     (stroke (width 0) (type default))
   )
-  (wire (pts (xy 180.34 64.77) (xy 180.34 54.61))
+  (wire (pts (xy 180.34 66.04) (xy 180.34 54.61))
     (stroke (width 0) (type default))
   )
@@
     (stroke (width 0) (type default))
   )
-  (wire (pts (xy 180.34 64.77) (xy 209.55 64.77))
+  (wire (pts (xy 180.34 66.04) (xy 209.55 66.04))
     (stroke (width 0) (type default))
   )
@@
     (stroke (width 0) (type default))
   )
-  (wire (pts (xy 185.42 60.96) (xy 185.42 59.69))
+  (wire (pts (xy 185.42 62.23) (xy 185.42 59.69))
     (stroke (width 0) (type default))
   )
@@
     (fill (type none))
   )
-  (text "Circuito Passa Faixas 2ª Ordem SK" (at 194.31 77.47 0)
+  (text "Circuito Passa Faixas 2ª Ordem SK" (at 199.39 78.74 0)
     (effects (font (size 1.27 1.27)) (justify left bottom))
   )
@@
     )
   )
-  (global_label "module -VCC" (shape input) (at 185.42 60.96 0) (fields_autoplaced)
+  (global_label "module -VCC" (shape input) (at 185.42 62.23 0) (fields_autoplaced)
     (effects (font (size 1.27 1.27)) (justify left))
-    (property "Intersheetrefs" "${INTERSHEET_REFS}" (at 203.645 60.96 0)
+    (property "Intersheetrefs" "${INTERSHEET_REFS}" (at 203.645 62.23 0)
       (effects (font (size 1.27 1.27)) (justify left) hide)
     )
@@
     )
   )
-  (symbol (lib_id "Device:R") (at 209.55 68.58 0) (mirror x) (unit 1)
-    (in_bom yes) (on_board yes) (dnp no)
-    (property "Reference" "R?" (at 213.36 69.85 90)
+  (symbol (lib_id "Device:R") (at 209.55 69.85 0) (mirror x) (unit 1)
+    (in_bom yes) (on_board yes) (dnp no)
+    (property "Reference" "R?" (at 212.09 68.58 90)
       (effects (font (size 1.27 1.27)) (justify left))
     )
-    (property "Value" "R" (at 213.36 67.31 90)
-      (effects (font (size 1.27 1.27)) (justify left) hide)
-    )
-    (property "Footprint" "Resistor_THT:R_Axial_DIN0207_L6.3mm_D2.5mm_P7.62mm_Horizontal" (at 207.772 68.58 90)
-      (effects (font (size 1.27 1.27)) hide)
-    )
-    (property "Datasheet" "~" (at 209.55 68.58 0)
+    (property "Value" "R" (at 213.36 68.58 90)
+      (effects (font (size 1.27 1.27)) (justify left) hide)
+    )
+    (property "Footprint" "Resistor_THT:R_Axial_DIN0207_L6.3mm_D2.5mm_P7.62mm_Horizontal" (at 207.772 69.85 90)
+      (effects (font (size 1.27 1.27)) hide)
+    )
+    (property "Datasheet" "~" (at 209.55 69.85 0)
       (effects (font (size 1.27 1.27)) hide)
     )
@@
     )
   )
-  (symbol (lib_id "power:PWR_FLAG") (at 185.42 59.69 90) (unit 1)
-    (in_bom yes) (on_board yes) (dnp no) (fields_autoplaced)
-    (property "Reference" "#FLG?" (at 183.515 59.69 0)
-      (effects (font (size 1.27 1.27)) hide)
-    )
-    (property "Value" "PWR_FLAG" (at 180.34 59.69 0)
-      (effects (font (size 1.27 1.27)) hide)
-    )
-    (property "Footprint" "" (at 185.42 59.69 0)
-      (effects (font (size 1.27 1.27)) hide)
-    )
-    (property "Datasheet" "~" (at 185.42 59.69 0)
-      (effects (font (size 1.27 1.27)) hide)
-    )
-    (pin "1")
-    (instances
-      (project "kicad"
-        (path "/1ce81232-195d-4047-8575-458c62622b55"
-          (reference "#FLG?") (unit 1)
-        )
-      )
-      (project "bandPassSecondOrderSK"
-        (path "/2121d978-39fd-4952-bc51-dbaf52d83413"
-          (reference "#FLG02") (unit 1)
-        )
-      )
-    )
-  )
-  (symbol (lib_id "power:PWR_FLAG") (at 185.42 44.45 90) (unit 1)
-    (in_bom yes) (on_board yes) (dnp no) (fields_autoplaced)
-    (property "Reference" "#FLG?" (at 183.515 44.45 0)
-      (effects (font (size 1.27 1.27)) hide)
-    )
-    (property "Value" "PWR_FLAG" (at 180.34 44.45 0)
-      (effects (font (size 1.27 1.27)) hide)
-    )
-    (property "Footprint" "" (at 185.42 44.45 0)
-      (effects (font (size 1.27 1.27)) hide)
-    )
-    (property "Datasheet" "~" (at 185.42 44.45 0)
-      (effects (font (size 1.27 1.27)) hide)
-    )
-    (pin "1")
-    (instances
-      (project "kicad"
-        (path "/1ce81232-195d-4047-8575-458c62622b55"
-          (reference "#FLG?") (unit 1)
-        )
-      )
-      (project "bandPassSecondOrderSK"
-        (path "/2121d978-39fd-4952-bc51-dbaf52d83413"
-          (reference "#FLG01") (unit 1)
-        )
-      )
-    )
-  )
   (symbol (lib_id "Connector:Conn_01x06_Pin") (at 233.68 66.04 0) (mirror y) (unit 1)
     (in_bom yes) (on_board yes) (dnp no)
@@
   (symbol (lib_id "Device:R") (at 209.55 57.15 0) (unit 1)
     (in_bom yes) (on_board yes) (dnp no)
-    (property "Reference" "R?" (at 212.09 55.88 0)
+    (property "Reference" "R?" (at 212.09 58.42 90)
       (effects (font (size 1.27 1.27)) (justify left))
     )
@@
     )
   )
-  (symbol (lib_id "power:GND") (at 209.55 72.39 0) (unit 1)
-    (in_bom yes) (on_board yes) (dnp no)
-    (property "Reference" "#PWR?" (at 209.55 78.74 0)
-      (effects (font (size 1.27 1.27)) hide)
-    )
-    (property "Value" "GND" (at 209.55 76.2 0)
-      (effects (font (size 1.27 1.27)) hide)
-    )
-    (property "Footprint" "" (at 209.55 72.39 0)
-      (effects (font (size 1.27 1.27)) hide)
-    )
-    (property "Datasheet" "" (at 209.55 72.39 0)
-      (effects (font (size 1.27 1.27)) hide)
-    )
+  (symbol (lib_id "power:GND") (at 209.55 73.66 0) (unit 1)
+    (in_bom yes) (on_board yes) (dnp no)
+    (property "Reference" "#PWR?" (at 209.55 80.01 0)
+      (effects (font (size 1.27 1.27)) hide)
+    )
+    (property "Value" "GND" (at 209.55 77.47 0)
+      (effects (font (size 1.27 1.27)) hide)
+    )
+    (property "Footprint" "" (at 209.55 73.66 0)
+      (effects (font (size 1.27 1.27)) hide)
+    )
+    (property "Datasheet" "" (at 209.55 73.66 0)
+      (effects (font (size 1.27 1.27)) hide)
+    )
