File: modules/differentiator/differentiator.kicad_sch (KiCad schematic)
At the start: 4 parts, among them J102 Conn_01x06_Pin, U102 TL071

Commit message: Little changes on each schematic
Changed lines of the file:
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@@
   (junction (at 137.16 78.74) (diameter 0) (color 0 0 0 0)
-  )
-  (junction (at 139.7 73.66) (diameter 0) (color 0 0 0 0)
   )
   (junction (at 132.08 88.9) (diameter 0) (color 0 0 0 0)
@@
     (stroke (width 0) (type default))
   )
+  (wire (pts (xy 144.78 86.36) (xy 144.78 83.82))
+    (stroke (width 0) (type default))
+  )
   (wire (pts (xy 130.81 88.9) (xy 132.08 88.9))
     (stroke (width 0) (type default))
@@
     )
   )
-  (global_label "module -VCC" (shape input) (at 144.78 83.82 0) (fields_autoplaced)
+  (global_label "module -VCC" (shape input) (at 144.78 86.36 0) (fields_autoplaced)
     (effects (font (size 1.27 1.27)) (justify left))
-    (property "Intersheetrefs" "${INTERSHEET_REFS}" (at 163.005 83.82 0)
+    (property "Intersheetrefs" "${INTERSHEET_REFS}" (at 163.005 86.36 0)
       (effects (font (size 1.27 1.27)) (justify left) hide)
     )
@@
     )
   )
-  (symbol (lib_id "power:PWR_FLAG") (at 139.7 73.66 0) (unit 1)
-    (in_bom yes) (on_board yes) (dnp no) (fields_autoplaced)
-    (property "Reference" "#FLG?" (at 139.7 71.755 0)
-      (effects (font (size 1.27 1.27)) hide)
-    )
-    (property "Value" "PWR_FLAG" (at 139.7 68.58 0)
-      (effects (font (size 1.27 1.27)) hide)
-    )
-    (property "Footprint" "" (at 139.7 73.66 0)
-      (effects (font (size 1.27 1.27)) hide)
-    )
-    (property "Datasheet" "~" (at 139.7 73.66 0)
-      (effects (font (size 1.27 1.27)) hide)
-    )
-    (pin "1")
-    (instances
-      (project "kicad"
-        (path "/1ce81232-195d-4047-8575-458c62622b55"
-          (reference "#FLG?") (unit 1)
-        )
-      )
-      (project "differentiator"
-        (path "/dfd7bb8f-212b-4fda-8920-38793b0fde80"
-          (reference "#FLG02") (unit 1)
-        )
-      )
-    )
-  )
   (symbol (lib_id "Connector:Conn_01x06_Pin") (at 186.69 86.36 0) (mirror y) (unit 1)
     (in_bom yes) (on_board yes) (dnp no)
@@
         )
       )
-    )
-  )
-  (symbol (lib_id "power:PWR_FLAG") (at 144.78 68.58 90) (unit 1)
-    (in_bom yes) (on_board yes) (dnp no) (fields_autoplaced)
-    (property "Reference" "#FLG?" (at 142.875 68.58 0)
-      (effects (font (size 1.27 1.27)) hide)
-    )
-    (property "Value" "PWR_FLAG" (at 139.7 68.58 0)
-      (effects (font (size 1.27 1.27)) hide)
-    )
-    (property "Footprint" "" (at 144.78 68.58 0)
-      (effects (font (size 1.27 1.27)) hide)
-    )
-    (property "Datasheet" "~" (at 144.78 68.58 0)
-      (effects (font (size 1.27 1.27)) hide)
-    )
-    (pin "1")
-    (instances
-      (project "kicad"
-        (path "/1ce81232-195d-4047-8575-458c62622b55"
-          (reference "#FLG?") (unit 1)
-        )
-      )
-      (project "differentiator"
-        (path "/dfd7bb8f-212b-4fda-8920-38793b0fde80"
-          (reference "#FLG01") (unit 1)
-        )
-      )
-    )
-  )
-  (symbol (lib_id "power:PWR_FLAG") (at 144.78 83.82 90) (unit 1)
-    (in_bom yes) (on_board yes) (dnp no) (fields_autoplaced)
-    (property "Reference" "#FLG?" (at 142.875 83.82 0)
-      (effects (font (size 1.27 1.27)) hide)
-    )
-    (property "Value" "PWR_FLAG" (at 139.7 83.82 0)
-      (effects (font (size 1.27 1.27)) hide)
-    )
-    (property "Footprint" "" (at 144.78 83.82 0)
-      (effects (font (size 1.27 1.27)) hide)
-    )
-    (property "Datasheet" "~" (at 144.78 83.82 0)
-      (effects (font (size 1.27 1.27)) hide)
-    )
-    (pin "1")
-    (instances
-      (project "kicad"
-        (path "/1ce81232-195d-4047-8575-458c62622b55"
-          (reference "#FLG?") (unit 1)
-        )
-      )
-      (project "differentiator"
-        (path "/dfd7bb8f-212b-4fda-8920-38793b0fde80"
-          (reference "#FLG03") (unit 1)
-        )
-      )
