File: modules/highPassFirstOrder/highPassFirstOrder.kicad_sch (KiCad schematic)
At the start: 5 parts

Commit message: Little changes on each schematic
Changed lines of the file:
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@@
   (junction (at 95.25 85.09) (diameter 0) (color 0 0 0 0)
-  )
-  (junction (at 102.87 77.47) (diameter 0) (color 0 0 0 0)
   )
   (junction (at 85.09 67.31) (diameter 0) (color 0 0 0 0)
@@
     (stroke (width 0) (type default))
   )
-  (wire (pts (xy 102.87 78.74) (xy 102.87 77.47))
+  (wire (pts (xy 102.87 80.01) (xy 102.87 77.47))
     (stroke (width 0) (type default))
   )
@@
     )
   )
-  (global_label "module -VCC" (shape input) (at 102.87 78.74 0) (fields_autoplaced)
+  (global_label "module -VCC" (shape input) (at 102.87 80.01 0) (fields_autoplaced)
     (effects (font (size 1.27 1.27)) (justify left))
-    (property "Intersheetrefs" "${INTERSHEET_REFS}" (at 121.095 78.74 0)
+    (property "Intersheetrefs" "${INTERSHEET_REFS}" (at 121.095 80.01 0)
       (effects (font (size 1.27 1.27)) (justify left) hide)
     )
@@
         (path "/393aa0ca-5eb7-4cb7-9410-c524d12d8676"
           (reference "C1") (unit 1)
-        )
-      )
-    )
-  )
-  (symbol (lib_id "power:PWR_FLAG") (at 102.87 77.47 90) (unit 1)
-    (in_bom yes) (on_board yes) (dnp no) (fields_autoplaced)
-    (property "Reference" "#FLG?" (at 100.965 77.47 0)
-      (effects (font (size 1.27 1.27)) hide)
-    )
-    (property "Value" "PWR_FLAG" (at 97.79 77.47 0)
-      (effects (font (size 1.27 1.27)) hide)
-    )
-    (property "Footprint" "" (at 102.87 77.47 0)
-      (effects (font (size 1.27 1.27)) hide)
-    )
-    (property "Datasheet" "~" (at 102.87 77.47 0)
-      (effects (font (size 1.27 1.27)) hide)
-    )
-    (pin "1")
-    (instances
-      (project "kicad"
-        (path "/1ce81232-195d-4047-8575-458c62622b55"
-          (reference "#FLG?") (unit 1)
-        )
-      )
-      (project "highPassFirstOrder"
-        (path "/393aa0ca-5eb7-4cb7-9410-c524d12d8676"
-          (reference "#FLG02") (unit 1)
         )
       )
@@
         )
       )
-    )
-  )
-  (symbol (lib_id "power:PWR_FLAG") (at 102.87 62.23 0) (unit 1)
-    (in_bom yes) (on_board yes) (dnp no) (fields_autoplaced)
-    (property "Reference" "#FLG?" (at 102.87 60.325 0)
-      (effects (font (size 1.27 1.27)) hide)
-    )
-    (property "Value" "PWR_FLAG" (at 102.87 57.15 0)
-      (effects (font (size 1.27 1.27)) hide)
-    )
-    (property "Footprint" "" (at 102.87 62.23 0)
-      (effects (font (size 1.27 1.27)) hide)
-    )
-    (property "Datasheet" "~" (at 102.87 62.23 0)
-      (effects (font (size 1.27 1.27)) hide)
-    )
-    (pin "1")
-    (instances
-      (project "kicad"
-        (path "/1ce81232-195d-4047-8575-458c62622b55"
-          (reference "#FLG?") (unit 1)
-        )
-      )
-      (project "highPassFirstOrder"
-        (path "/393aa0ca-5eb7-4cb7-9410-c524d12d8676"
-          (reference "#FLG01") (unit 1)
-        )
-      )
