File: modules/highPassSecondOrderSK/highPassSecondOrderSK.kicad_sch (KiCad schematic)
At the start: 8 parts

Commit message: Update moudules
Parts:
- removed C? (x2): C, symbol Device:C
- removed R? (x3): R, Resistor_THT:R_Axial_DIN0207_L6.3mm_D2.5mm_P7.62mm_Horizontal, symbol Device:R
- added C? (x2): C, symbol Device:C
- added R? (x3): R, Resistor_THT:R_Axial_DIN0207_L6.3mm_D2.5mm_P7.62mm_Horizontal, symbol Device:R
Connections:
- net GND: now also R?.1, R?.2
- net module Out: now also R?.2
- net module in 1: now also C?.1
- net at U?.2 (-): now also R?.2, R?.2
- net at U?.3 (+): now also C?.2, R?.1
- new net: C?.1, C?.2, R?.1

Commit message: Little changes on each schematic
Other:
- note added: "Circuito Passa Altas 2ª Ordem SK"
- note removed: "Circuito Passa Baixas 2ª Ordem SK"
- moved on the sheet: R?
Changed lines of the file:
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@@
   (junction (at 162.56 82.55) (diameter 0) (color 0 0 0 0)
   )
-  (junction (at 162.56 95.25) (diameter 0) (color 0 0 0 0)
-  )
   (junction (at 158.75 82.55) (diameter 0) (color 0 0 0 0)
   )
@@
   (junction (at 118.11 90.17) (diameter 0) (color 0 0 0 0)
   )
-  (junction (at 138.43 90.17) (diameter 0) (color 0 0 0 0)
+  (junction (at 162.56 96.52) (diameter 0) (color 0 0 0 0)
   )
   (junction (at 118.11 78.74) (diameter 0) (color 0 0 0 0)
@@
     (stroke (width 0) (type default))
   )
-  (wire (pts (xy 133.35 95.25) (xy 133.35 85.09))
+  (wire (pts (xy 133.35 96.52) (xy 133.35 85.09))
     (stroke (width 0) (type default))
   )
@@
     (stroke (width 0) (type default))
   )
-  (wire (pts (xy 138.43 91.44) (xy 138.43 90.17))
-    (stroke (width 0) (type default))
-  )
-  (wire (pts (xy 133.35 95.25) (xy 162.56 95.25))
+  (wire (pts (xy 138.43 92.71) (xy 138.43 90.17))
+    (stroke (width 0) (type default))
+  )
+  (wire (pts (xy 133.35 96.52) (xy 162.56 96.52))
     (stroke (width 0) (type default))
   )
@@
     (stroke (width 0) (type default))
   )
-  (wire (pts (xy 162.56 95.25) (xy 162.56 91.44))
-    (stroke (width 0) (type default))
-  )
   (wire (pts (xy 118.11 90.17) (xy 118.11 102.87))
     (stroke (width 0) (type default))
@@
   )
   (wire (pts (xy 129.54 80.01) (xy 133.35 80.01))
+    (stroke (width 0) (type default))
+  )
+  (wire (pts (xy 162.56 91.44) (xy 162.56 96.52))
     (stroke (width 0) (type default))
   )
@@
     (fill (type none))
   )
-  (text "Circuito Passa Baixas 2ª Ordem SK" (at 154.94 109.22 0)
+  (text "Circuito Passa Altas 2ª Ordem SK" (at 154.94 109.22 0)
     (effects (font (size 1.27 1.27)) (justify left bottom))
   )
@@
     )
   )
-  (global_label "module -VCC" (shape input) (at 138.43 91.44 0) (fields_autoplaced)
+  (global_label "module -VCC" (shape input) (at 138.43 92.71 0) (fields_autoplaced)
     (effects (font (size 1.27 1.27)) (justify left))
-    (property "Intersheetrefs" "${INTERSHEET_REFS}" (at 156.655 91.44 0)
+    (property "Intersheetrefs" "${INTERSHEET_REFS}" (at 156.655 92.71 0)
       (effects (font (size 1.27 1.27)) (justify left) hide)
     )
@@
     (property "Intersheetrefs" "${INTERSHEET_REFS}" (at 156.655 74.93 0)
       (effects (font (size 1.27 1.27)) (justify left) hide)
-    )
-  )
-  (symbol (lib_id "power:PWR_FLAG") (at 138.43 90.17 90) (unit 1)
-    (in_bom yes) (on_board yes) (dnp no) (fields_autoplaced)
-    (property "Reference" "#FLG?" (at 136.525 90.17 0)
-      (effects (font (size 1.27 1.27)) hide)
-    )
-    (property "Value" "PWR_FLAG" (at 133.35 90.17 0)
-      (effects (font (size 1.27 1.27)) hide)
-    )
-    (property "Footprint" "" (at 138.43 90.17 0)
-      (effects (font (size 1.27 1.27)) hide)
-    )
-    (property "Datasheet" "~" (at 138.43 90.17 0)
-      (effects (font (size 1.27 1.27)) hide)
-    )
-    (pin "1")
-    (instances
-      (project "kicad"
-        (path "/1ce81232-195d-4047-8575-458c62622b55"
-          (reference "#FLG?") (unit 1)
-        )
-      )
-      (project "highPassSecondOrderSK"
-        (path "/4f83be14-7577-43b1-af42-d25b34c97057"
-          (reference "#FLG02") (unit 1)
-        )
-      )
     )
   )
@@
     )
   )
-  (symbol (lib_id "Device:R") (at 162.56 99.06 0) (mirror x) (unit 1)
-    (in_bom yes) (on_board yes) (dnp no)
-    (property "Reference" "R?" (at 166.37 100.33 90)
+  (symbol (lib_id "Device:R") (at 162.56 100.33 0) (mirror x) (unit 1)
+    (in_bom yes) (on_board yes) (dnp no)
+    (property "Reference" "R?" (at 166.37 101.6 90)
       (effects (font (size 1.27 1.27)) (justify left))
     )
-    (property "Value" "R" (at 166.37 97.79 90)
-      (effects (font (size 1.27 1.27)) (justify left) hide)
-    )
-    (property "Footprint" "Resistor_THT:R_Axial_DIN0207_L6.3mm_D2.5mm_P7.62mm_Horizontal" (at 160.782 99.06 90)
-      (effects (font (size 1.27 1.27)) hide)
-    )
-    (property "Datasheet" "~" (at 162.56 99.06 0)
+    (property "Value" "R" (at 166.37 99.06 90)
+      (effects (font (size 1.27 1.27)) (justify left) hide)
+    )
+    (property "Footprint" "Resistor_THT:R_Axial_DIN0207_L6.3mm_D2.5mm_P7.62mm_Horizontal" (at 160.782 100.33 90)
+      (effects (font (size 1.27 1.27)) hide)
+    )
+    (property "Datasheet" "~" (at 162.56 100.33 0)
       (effects (font (size 1.27 1.27)) hide)
     )
@@
     )
   )
-  (symbol (lib_id "power:PWR_FLAG") (at 138.43 74.93 90) (unit 1)
-    (in_bom yes) (on_board yes) (dnp no) (fields_autoplaced)
-    (property "Reference" "#FLG?" (at 136.525 74.93 0)
-      (effects (font (size 1.27 1.27)) hide)
-    )
-    (property "Value" "PWR_FLAG" (at 133.35 74.93 0)
-      (effects (font (size 1.27 1.27)) hide)
-    )
-    (property "Footprint" "" (at 138.43 74.93 0)
-      (effects (font (size 1.27 1.27)) hide)
-    )
-    (property "Datasheet" "~" (at 138.43 74.93 0)
-      (effects (font (size 1.27 1.27)) hide)
-    )
-    (pin "1")
-    (instances
-      (project "kicad"
-        (path "/1ce81232-195d-4047-8575-458c62622b55"
-          (reference "#FLG?") (unit 1)
-        )
-      )
-      (project "highPassSecondOrderSK"
-        (path "/4f83be14-7577-43b1-af42-d25b34c97057"
-          (reference "#FLG01") (unit 1)
-        )
-      )
-    )
-  )
   (symbol (lib_id "power:GND") (at 129.54 99.06 0) (unit 1)
     (in_bom yes) (on_board yes) (dnp no)
@@
     )
   )
-  (symbol (lib_id "power:GND") (at 162.56 102.87 0) (unit 1)
-    (in_bom yes) (on_board yes) (dnp no)
-    (property "Reference" "#PWR?" (at 162.56 109.22 0)
-      (effects (font (size 1.27 1.27)) hide)
-    )
-    (property "Value" "GND" (at 162.56 106.68 0)
-      (effects (font (size 1.27 1.27)) hide)
-    )
-    (property "Footprint" "" (at 162.56 102.87 0)
-      (effects (font (size 1.27 1.27)) hide)
-    )
-    (property "Datasheet" "" (at 162.56 102.87 0)
-      (effects (font (size 1.27 1.27)) hide)
-    )
+  (symbol (lib_id "power:GND") (at 162.56 104.14 0) (unit 1)
+    (in_bom yes) (on_board yes) (dnp no)
+    (property "Reference" "#PWR?" (at 162.56 110.49 0)
+      (effects (font (size 1.27 1.27)) hide)
+    )
+    (property "Value" "GND" (at 162.56 107.95 0)
+      (effects (font (size 1.27 1.27)) hide)
+    )
+    (property "Footprint" "" (at 162.56 104.14 0)
+      (effects (font (size 1.27 1.27)) hide)
+    )
+    (property "Datasheet" "" (at 162.56 104.14 0)
+      (effects (font (size 1.27 1.27)) hide)
+    )
