File: modules/integrator/integrator.kicad_sch (KiCad schematic)
At the start: 4 parts

Commit message: Little changes on each schematic
Changed lines of the file:
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@@
+    (stroke (width 0) (type default))
+  )
+  (wire (pts (xy 144.78 102.87) (xy 144.78 100.33))
     (stroke (width 0) (type default))
   )
@@
     )
   )
-  (global_label "module -VCC" (shape input) (at 144.78 100.33 0) (fields_autoplaced)
+  (global_label "module -VCC" (shape input) (at 144.78 102.87 0) (fields_autoplaced)
     (effects (font (size 1.27 1.27)) (justify left))
-    (property "Intersheetrefs" "${INTERSHEET_REFS}" (at 160.8279 100.33 0)
+    (property "Intersheetrefs" "${INTERSHEET_REFS}" (at 160.8279 102.87 0)
       (effects (font (size 1.27 1.27)) (justify left) hide)
     )
@@
         )
       )
-    )
-  )
-  (symbol (lib_id "power:PWR_FLAG") (at 144.78 85.09 90) (unit 1)
-    (in_bom yes) (on_board yes) (dnp no) (fields_autoplaced)
-    (property "Reference" "#FLG?" (at 142.875 85.09 0)
-      (effects (font (size 1.27 1.27)) hide)
-    )
-    (property "Value" "PWR_FLAG" (at 139.7 85.09 0)
-      (effects (font (size 1.27 1.27)) hide)
-    )
-    (property "Footprint" "" (at 144.78 85.09 0)
-      (effects (font (size 1.27 1.27)) hide)
-    )
-    (property "Datasheet" "~" (at 144.78 85.09 0)
-      (effects (font (size 1.27 1.27)) hide)
-    )
-    (pin "1")
-    (instances
-      (project "kicad"
-        (path "/1ce81232-195d-4047-8575-458c62622b55"
-          (reference "#FLG?") (unit 1)
-        )
-      )
-      (project "integrator"
-        (path "/79e45918-4032-45ce-9400-3d5c85238198"
-          (reference "#FLG01") (unit 1)
-        )
-      )
-    )
-  )
-  (symbol (lib_id "power:PWR_FLAG") (at 144.78 100.33 90) (unit 1)
-    (in_bom yes) (on_board yes) (dnp no) (fields_autoplaced)
-    (property "Reference" "#FLG?" (at 142.875 100.33 0)
-      (effects (font (size 1.27 1.27)) hide)
-    )
-    (property "Value" "PWR_FLAG" (at 139.7 100.33 0)
-      (effects (font (size 1.27 1.27)) hide)
-    )
-    (property "Footprint" "" (at 144.78 100.33 0)
-      (effects (font (size 1.27 1.27)) hide)
-    )
-    (property "Datasheet" "~" (at 144.78 100.33 0)
-      (effects (font (size 1.27 1.27)) hide)
-    )
-    (pin "1")
-    (instances
-      (project "kicad"
-        (path "/1ce81232-195d-4047-8575-458c62622b55"
-          (reference "#FLG?") (unit 1)
-        )
-      )
-      (project "integrator"
-        (path "/79e45918-4032-45ce-9400-3d5c85238198"
-          (reference "#FLG02") (unit 1)
-        )
-      )
