File: modules/inversor/inversor.kicad_sch (KiCad schematic)
At the start: 4 parts, among them J1 Conn_01x06_Pin, U1 TL071

Commit message: Little changes on each schematic
Changed lines of the file:
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@@
   (junction (at 127 85.09) (diameter 0) (color 0 0 0 0)
-  )
-  (junction (at 134.62 90.17) (diameter 0) (color 0 0 0 0)
   )
   (junction (at 146.05 82.55) (diameter 0) (color 0 0 0 0)
@@
     (stroke (width 0) (type default))
   )
-  (wire (pts (xy 134.62 91.44) (xy 134.62 90.17))
+  (wire (pts (xy 134.62 92.71) (xy 134.62 90.17))
     (stroke (width 0) (type default))
   )
@@
     )
   )
-  (global_label "module -VCC" (shape input) (at 134.62 91.44 0) (fields_autoplaced)
+  (global_label "module -VCC" (shape input) (at 134.62 92.71 0) (fields_autoplaced)
     (effects (font (size 1.27 1.27)) (justify left))
-    (property "Intersheetrefs" "${INTERSHEET_REFS}" (at 150.6679 91.44 0)
+    (property "Intersheetrefs" "${INTERSHEET_REFS}" (at 150.6679 92.71 0)
       (effects (font (size 1.27 1.27)) (justify left) hide)
     )
@@
         )
       )
-    )
-  )
-  (symbol (lib_id "power:PWR_FLAG") (at 134.62 74.93 90) (unit 1)
-    (in_bom yes) (on_board yes) (dnp no) (fields_autoplaced)
-    (property "Reference" "#FLG?" (at 132.715 74.93 0)
-      (effects (font (size 1.27 1.27)) hide)
-    )
-    (property "Value" "PWR_FLAG" (at 129.54 74.93 0)
-      (effects (font (size 1.27 1.27)) hide)
-    )
-    (property "Footprint" "" (at 134.62 74.93 0)
-      (effects (font (size 1.27 1.27)) hide)
-    )
-    (property "Datasheet" "~" (at 134.62 74.93 0)
-      (effects (font (size 1.27 1.27)) hide)
-    )
-    (pin "1")
-    (instances
-      (project "kicad"
-        (path "/1ce81232-195d-4047-8575-458c62622b55"
-          (reference "#FLG?") (unit 1)
-        )
-      )
-      (project "inversor"
-        (path "/79fad7f2-24c3-4188-bddd-924ce12807be"
-          (reference "#FLG01") (unit 1)
-        )
-      )
-    )
-  )
-  (symbol (lib_id "power:PWR_FLAG") (at 134.62 90.17 90) (unit 1)
-    (in_bom yes) (on_board yes) (dnp no) (fields_autoplaced)
-    (property "Reference" "#FLG?" (at 132.715 90.17 0)
-      (effects (font (size 1.27 1.27)) hide)
-    )
-    (property "Value" "PWR_FLAG" (at 129.54 90.17 0)
-      (effects (font (size 1.27 1.27)) hide)
-    )
-    (property "Footprint" "" (at 134.62 90.17 0)
-      (effects (font (size 1.27 1.27)) hide)
-    )
-    (property "Datasheet" "~" (at 134.62 90.17 0)
-      (effects (font (size 1.27 1.27)) hide)
-    )
-    (pin "1")
-    (instances
-      (project "kicad"
-        (path "/1ce81232-195d-4047-8575-458c62622b55"
-          (reference "#FLG?") (unit 1)
-        )
-      )
-      (project "inversor"
-        (path "/79fad7f2-24c3-4188-bddd-924ce12807be"
-          (reference "#FLG02") (unit 1)
-        )
-      )
