File: modules/lowPassFirstOrder/lowPassFirstOrder.kicad_sch (KiCad schematic)
At the start: 5 parts

Commit message: Little changes on each schematic
Other:
- moved on the sheet: C?
Changed lines of the file:
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@@
   (junction (at 121.92 81.28) (diameter 0) (color 0 0 0 0)
   )
-  (junction (at 140.97 91.44) (diameter 0) (color 0 0 0 0)
-  )
   (junction (at 113.03 80.01) (diameter 0) (color 0 0 0 0)
   )
   (junction (at 140.97 78.74) (diameter 0) (color 0 0 0 0)
   )
-  (junction (at 129.54 86.36) (diameter 0) (color 0 0 0 0)
-  )
-  (junction (at 121.92 91.44) (diameter 0) (color 0 0 0 0)
+  (junction (at 121.92 93.98) (diameter 0) (color 0 0 0 0)
+  )
+  (junction (at 140.97 93.98) (diameter 0) (color 0 0 0 0)
   )
   (no_connect (at 132.08 86.36))
   (no_connect (at 134.62 86.36))
-  (wire (pts (xy 121.92 81.28) (xy 121.92 91.44))
-    (stroke (width 0) (type default))
-  )
-  (wire (pts (xy 140.97 91.44) (xy 140.97 78.74))
-    (stroke (width 0) (type default))
-  )
-  (wire (pts (xy 135.89 91.44) (xy 140.97 91.44))
+  (wire (pts (xy 140.97 93.98) (xy 140.97 100.33))
+    (stroke (width 0) (type default))
+  )
+  (wire (pts (xy 135.89 93.98) (xy 140.97 93.98))
     (stroke (width 0) (type default))
   )
@@
     (stroke (width 0) (type default))
   )
+  (wire (pts (xy 121.92 93.98) (xy 121.92 100.33))
+    (stroke (width 0) (type default))
+  )
   (wire (pts (xy 113.03 76.2) (xy 113.03 80.01))
     (stroke (width 0) (type default))
   )
-  (wire (pts (xy 129.54 87.63) (xy 129.54 86.36))
+  (wire (pts (xy 129.54 88.9) (xy 129.54 86.36))
     (stroke (width 0) (type default))
   )
@@
     (stroke (width 0) (type default))
   )
-  (wire (pts (xy 121.92 91.44) (xy 121.92 100.33))
+  (wire (pts (xy 121.92 81.28) (xy 121.92 93.98))
     (stroke (width 0) (type default))
   )
@@
     (stroke (width 0) (type default))
   )
-  (wire (pts (xy 140.97 91.44) (xy 140.97 100.33))
+  (wire (pts (xy 140.97 78.74) (xy 140.97 93.98))
     (stroke (width 0) (type default))
   )
@@
     (stroke (width 0) (type default))
   )
-  (wire (pts (xy 121.92 91.44) (xy 128.27 91.44))
+  (wire (pts (xy 121.92 93.98) (xy 128.27 93.98))
     (stroke (width 0) (type default))
   )
@@
     )
   )
-  (global_label "module -VCC" (shape input) (at 129.54 87.63 0) (fields_autoplaced)
+  (global_label "module -VCC" (shape input) (at 129.54 88.9 0) (fields_autoplaced)
     (effects (font (size 1.27 1.27)) (justify left))
-    (property "Intersheetrefs" "${INTERSHEET_REFS}" (at 147.765 87.63 0)
+    (property "Intersheetrefs" "${INTERSHEET_REFS}" (at 147.765 88.9 0)
       (effects (font (size 1.27 1.27)) (justify left) hide)
     )
@@
   (symbol (lib_id "Device:R") (at 132.08 100.33 270) (unit 1)
     (in_bom yes) (on_board yes) (dnp no)
-    (property "Reference" "R?" (at 133.35 102.87 90)
+    (property "Reference" "R?" (at 130.81 102.87 90)
       (effects (font (size 1.27 1.27)) (justify left))
     )
@@
         (path "/4e2f95ff-f3bc-46ec-8757-d1dd7a33cb35"
           (reference "R2") (unit 1)
-        )
-      )
-    )
-  )
-  (symbol (lib_id "power:PWR_FLAG") (at 129.54 86.36 90) (unit 1)
-    (in_bom yes) (on_board yes) (dnp no) (fields_autoplaced)
-    (property "Reference" "#FLG?" (at 127.635 86.36 0)
-      (effects (font (size 1.27 1.27)) hide)
-    )
-    (property "Value" "PWR_FLAG" (at 124.46 86.36 0)
-      (effects (font (size 1.27 1.27)) hide)
-    )
-    (property "Footprint" "" (at 129.54 86.36 0)
-      (effects (font (size 1.27 1.27)) hide)
-    )
-    (property "Datasheet" "~" (at 129.54 86.36 0)
-      (effects (font (size 1.27 1.27)) hide)
-    )
-    (pin "1")
-    (instances
-      (project "kicad"
-        (path "/1ce81232-195d-4047-8575-458c62622b55"
-          (reference "#FLG?") (unit 1)
-        )
-      )
-      (project "lowPassFirstOrder"
-        (path "/4e2f95ff-f3bc-46ec-8757-d1dd7a33cb35"
-          (reference "#FLG02") (unit 1)
         )
       )
@@
     )
   )
-  (symbol (lib_id "Device:C") (at 132.08 91.44 270) (unit 1)
+  (symbol (lib_id "Device:C") (at 132.08 93.98 270) (unit 1)
     (in_bom yes) (on_board yes) (dnp no)
     (property "Reference" "C?" (at 132.08 97.79 90)
       (effects (font (size 1.27 1.27)))
     )
-    (property "Value" "C" (at 132.08 95.25 90)
-      (effects (font (size 1.27 1.27)) hide)
-    )
-    (property "Footprint" "" (at 128.27 92.4052 0)
-      (effects (font (size 1.27 1.27)) hide)
-    )
-    (property "Datasheet" "~" (at 132.08 91.44 0)
+    (property "Value" "C" (at 132.08 97.79 90)
+      (effects (font (size 1.27 1.27)) hide)
+    )
+    (property "Footprint" "" (at 128.27 94.9452 0)
+      (effects (font (size 1.27 1.27)) hide)
+    )
+    (property "Datasheet" "~" (at 132.08 93.98 0)
       (effects (font (size 1.27 1.27)) hide)
     )
@@
         )
       )
-    )
-  )
-  (symbol (lib_id "power:PWR_FLAG") (at 129.54 71.12 90) (unit 1)
-    (in_bom yes) (on_board yes) (dnp no) (fields_autoplaced)
-    (property "Reference" "#FLG?" (at 127.635 71.12 0)
-      (effects (font (size 1.27 1.27)) hide)
-    )
-    (property "Value" "PWR_FLAG" (at 124.46 71.12 0)
-      (effects (font (size 1.27 1.27)) hide)
-    )
-    (property "Footprint" "" (at 129.54 71.12 0)
-      (effects (font (size 1.27 1.27)) hide)
-    )
-    (property "Datasheet" "~" (at 129.54 71.12 0)
-      (effects (font (size 1.27 1.27)) hide)
-    )
-    (pin "1")
-    (instances
-      (project "kicad"
-        (path "/1ce81232-195d-4047-8575-458c62622b55"
-          (reference "#FLG?") (unit 1)
-        )
-      )
-      (project "lowPassFirstOrder"
-        (path "/4e2f95ff-f3bc-46ec-8757-d1dd7a33cb35"
-          (reference "#FLG01") (unit 1)
-        )
-      )
