File: modules/lowPassSecondOrderSK/lowPassSecondOrderSK.kicad_sch (KiCad schematic)
At the start: 8 parts, among them J5 Conn_01x06_Pin, U6 TL071

Commit message: Update moudules
Parts:
- removed R14: R, Resistor_THT:R_Axial_DIN0207_L6.3mm_D2.5mm_P7.62mm_Horizontal, symbol Device:R
- added R4: R, Resistor_THT:R_Axial_DIN0207_L6.3mm_D2.5mm_P7.62mm_Horizontal, symbol Device:R
- renumbered C6 to C1, C7 to C2, J5 to J1, R9 to R1, R13 to R2, R11 to R3, U6 to U1
Connections:
- net GND: now also R4.1
- net at U1.2 (-): now also R3.2, R4.2
Changed lines of the file:
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@@
   (junction (at 139.7 69.85) (diameter 0) (color 0 0 0 0)
+  )
+  (junction (at 172.72 74.93) (diameter 0) (color 0 0 0 0)
   )
   (junction (at 128.27 58.42) (diameter 0) (color 0 0 0 0)
@@
     (stroke (width 0) (type default))
   )
-  (wire (pts (xy 165.1 74.93) (xy 172.72 74.93))
-    (stroke (width 0) (type default))
-  )
   (wire (pts (xy 148.59 82.55) (xy 168.91 82.55))
     (stroke (width 0) (type default))
@@
     (stroke (width 0) (type default))
   )
-  (wire (pts (xy 157.48 74.93) (xy 143.51 74.93))
+  (wire (pts (xy 143.51 74.93) (xy 172.72 74.93))
     (stroke (width 0) (type default))
   )
@@
   (symbol (lib_id "power:GND") (at 139.7 78.74 0) (unit 1)
     (in_bom yes) (on_board yes) (dnp no)
-    (property "Reference" "#PWR014" (at 139.7 85.09 0)
+    (property "Reference" "#PWR01" (at 139.7 85.09 0)
       (effects (font (size 1.27 1.27)) hide)
     )
@@
       (project "lowPassSecondOrderSK"
         (path "/1abb811e-e6a2-481c-ab83-294d796176de"
-          (reference "#PWR014") (unit 1)
+          (reference "#PWR01") (unit 1)
         )
       )
@@
   (symbol (lib_id "power:PWR_FLAG") (at 148.59 69.85 90) (unit 1)
     (in_bom yes) (on_board yes) (dnp no) (fields_autoplaced)
-    (property "Reference" "#FLG014" (at 146.685 69.85 0)
+    (property "Reference" "#FLG02" (at 146.685 69.85 0)
       (effects (font (size 1.27 1.27)) hide)
     )
@@
       (project "lowPassSecondOrderSK"
         (path "/1abb811e-e6a2-481c-ab83-294d796176de"
-          (reference "#FLG014") (unit 1)
+          (reference "#FLG02") (unit 1)
         )
       )
@@
   (symbol (lib_id "Amplifier_Operational:TL071") (at 151.13 62.23 0) (unit 1)
     (in_bom yes) (on_board yes) (dnp no) (fields_autoplaced)
-    (property "Reference" "U6" (at 160.02 58.0391 0)
+    (property "Reference" "U1" (at 160.02 58.0391 0)
       (effects (font (size 1.27 1.27)))
     )
@@
       (project "lowPassSecondOrderSK"
         (path "/1abb811e-e6a2-481c-ab83-294d796176de"
-          (reference "U6") (unit 1)
+          (reference "U1") (unit 1)
         )
       )
@@
   (symbol (lib_id "power:PWR_FLAG") (at 148.59 54.61 90) (unit 1)
     (in_bom yes) (on_board yes) (dnp no) (fields_autoplaced)
-    (property "Reference" "#FLG011" (at 146.685 54.61 0)
+    (property "Reference" "#FLG01" (at 146.685 54.61 0)
       (effects (font (size 1.27 1.27)) hide)
     )
@@
       (project "lowPassSecondOrderSK"
         (path "/1abb811e-e6a2-481c-ab83-294d796176de"
-          (reference "#FLG011") (unit 1)
+          (reference "#FLG01") (unit 1)
         )
       )
@@
     )
   )
-  (symbol (lib_id "Device:R") (at 161.29 74.93 90) (mirror x) (unit 1)
-    (in_bom yes) (on_board yes) (dnp no)
-    (property "Reference" "R14" (at 160.02 78.74 90)
+  (symbol (lib_id "Device:R") (at 172.72 78.74 0) (mirror x) (unit 1)
+    (in_bom yes) (on_board yes) (dnp no)
+    (property "Reference" "R4" (at 176.53 80.01 90)
       (effects (font (size 1.27 1.27)) (justify left))
     )
-    (property "Value" "R" (at 162.56 78.74 90)
-      (effects (font (size 1.27 1.27)) (justify left) hide)
-    )
-    (property "Footprint" "Resistor_THT:R_Axial_DIN0207_L6.3mm_D2.5mm_P7.62mm_Horizontal" (at 161.29 73.152 90)
-      (effects (font (size 1.27 1.27)) hide)
-    )
-    (property "Datasheet" "~" (at 161.29 74.93 0)
-      (effects (font (size 1.27 1.27)) hide)
-    )
-    (pin "1")
-    (pin "2")
-    (instances
-      (project "lowPassSecondOrderSK"
-        (path "/1abb811e-e6a2-481c-ab83-294d796176de"
-          (reference "R14") (unit 1)
+    (property "Value" "R" (at 176.53 77.47 90)
+      (effects (font (size 1.27 1.27)) (justify left) hide)
+    )
+    (property "Footprint" "Resistor_THT:R_Axial_DIN0207_L6.3mm_D2.5mm_P7.62mm_Horizontal" (at 170.942 78.74 90)
+      (effects (font (size 1.27 1.27)) hide)
+    )
+    (property "Datasheet" "~" (at 172.72 78.74 0)
+      (effects (font (size 1.27 1.27)) hide)
+    )
+    (pin "1")
+    (pin "2")
+    (instances
+      (project "lowPassSecondOrderSK"
+        (path "/1abb811e-e6a2-481c-ab83-294d796176de"
+          (reference "R4") (unit 1)
         )
       )
@@
   (symbol (lib_id "power:GND") (at 194.31 76.2 270) (unit 1)
     (in_bom yes) (on_board yes) (dnp no) (fields_autoplaced)
-    (property "Reference" "#PWR011" (at 187.96 76.2 0)
+    (property "Reference" "#PWR03" (at 187.96 76.2 0)
       (effects (font (size 1.27 1.27)) hide)
     )
@@
       (project "lowPassSecondOrderSK"
         (path "/1abb811e-e6a2-481c-ab83-294d796176de"
-          (reference "#PWR011") (unit 1)
+          (reference "#PWR03") (unit 1)
         )
       )
@@
   (symbol (lib_id "Device:R") (at 132.08 69.85 90) (mirror x) (unit 1)
     (in_bom yes) (on_board yes) (dnp no)
-    (property "Reference" "R13" (at 130.81 71.12 0)
+    (property "Reference" "R2" (at 130.81 71.12 0)
       (effects (font (size 1.27 1.27)) (justify left))
     )
@@
       (project "lowPassSecondOrderSK"
         (path "/1abb811e-e6a2-481c-ab83-294d796176de"
-          (reference "R13") (unit 1)
+          (reference "R2") (unit 1)
         )
       )
@@
   (symbol (lib_id "Device:R") (at 172.72 67.31 0) (unit 1)
     (in_bom yes) (on_board yes) (dnp no)
-    (property "Reference" "R11" (at 175.26 66.04 0)
+    (property "Reference" "R3" (at 175.26 66.04 0)
       (effects (font (size 1.27 1.27)) (justify left))
     )
@@
       (project "lowPassSecondOrderSK"
         (path "/1abb811e-e6a2-481c-ab83-294d796176de"
-          (reference "R11") (unit 1)
+          (reference "R3") (unit 1)
         )
       )
@@
   (symbol (lib_id "Connector:Conn_01x06_Pin") (at 199.39 76.2 0) (mirror y) (unit 1)
     (in_bom yes) (on_board yes) (dnp no)
-    (property "Reference" "J5" (at 198.755 66.04 0)
+    (property "Reference" "J1" (at 198.755 66.04 0)
       (effects (font (size 1.27 1.27)) hide)
     )
@@
       (project "lowPassSecondOrderSK"
         (path "/1abb811e-e6a2-481c-ab83-294d796176de"
-          (reference "J5") (unit 1)
+          (reference "J1") (unit 1)
         )
       )
@@
   (symbol (lib_id "Device:C") (at 139.7 74.93 0) (unit 1)
     (in_bom yes) (on_board yes) (dnp no)
-    (property "Reference" "C6" (at 135.89 72.39 90)
+    (property "Reference" "C1" (at 135.89 72.39 90)
       (effects (font (size 1.27 1.27)))
     )
@@
       (project "lowPassSecondOrderSK"
         (path "/1abb811e-e6a2-481c-ab83-294d796176de"
-          (reference "C6") (unit 1)
+          (reference "C1") (unit 1)
         )
       )
@@
   (symbol (lib_id "Device:R") (at 128.27 64.77 0) (unit 1)
     (in_bom yes) (on_board yes) (dnp no)
-    (property "Reference" "R9" (at 129.54 63.5 0)
+    (property "Reference" "R1" (at 129.54 63.5 0)
       (effects (font (size 1.27 1.27)) (justify left))
     )
@@
       (project "lowPassSecondOrderSK"
         (path "/1abb811e-e6a2-481c-ab83-294d796176de"
-          (reference "R9") (unit 1)
+          (reference "R1") (unit 1)
         )
       )
@@
     )
   )
+  (symbol (lib_id "power:GND") (at 172.72 82.55 0) (unit 1)
+    (in_bom yes) (on_board yes) (dnp no)
+    (property "Reference" "#PWR02" (at 172.72 88.9 0)
+      (effects (font (size 1.27 1.27)) hide)
+    )
+    (property "Value" "GND" (at 172.72 86.36 0)
+      (effects (font (size 1.27 1.27)) hide)
+    )
+    (property "Footprint" "" (at 172.72 82.55 0)
+      (effects (font (size 1.27 1.27)) hide)
+    )
+    (property "Datasheet" "" (at 172.72 82.55 0)
+      (effects (font (size 1.27 1.27)) hide)
+    )
+    (pin "1")
+    (instances
+      (project "lowPassSecondOrderSK"
+        (path "/1abb811e-e6a2-481c-ab83-294d796176de"
+          (reference "#PWR02") (unit 1)
+        )
+      )
+      (project "kicad"
+        (path "/1ce81232-195d-4047-8575-458c62622b55"
+          (reference "#PWR?") (unit 1)
+        )
+      )
+    )
+  )
   (symbol (lib_id "Device:C") (at 144.78 82.55 90) (unit 1)
     (in_bom yes) (on_board yes) (dnp no)
-    (property "Reference" "C7" (at 142.24 86.36 90)
+    (property "Reference" "C2" (at 142.24 86.36 90)
       (effects (font (size 1.27 1.27)))
     )
@@
       (project "lowPassSecondOrderSK"
         (path "/1abb811e-e6a2-481c-ab83-294d796176de"
-          (reference "C7") (unit 1)
-        )
-      )
+          (reference "C2") (unit 1)
+        )
+      )

Commit message: Little changes on each schematic
Other:
- moved on the sheet: R4
Changed lines of the file:
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@@
   (junction (at 139.7 69.85) (diameter 0) (color 0 0 0 0)
   )
-  (junction (at 172.72 74.93) (diameter 0) (color 0 0 0 0)
-  )
   (junction (at 128.27 58.42) (diameter 0) (color 0 0 0 0)
   )
   (junction (at 168.91 62.23) (diameter 0) (color 0 0 0 0)
   )
-  (junction (at 148.59 69.85) (diameter 0) (color 0 0 0 0)
+  (junction (at 172.72 76.2) (diameter 0) (color 0 0 0 0)
   )
   (no_connect (at 153.67 69.85))
@@
     (stroke (width 0) (type default))
   )
-  (wire (pts (xy 148.59 71.12) (xy 148.59 69.85))
+  (wire (pts (xy 148.59 72.39) (xy 148.59 69.85))
     (stroke (width 0) (type default))
   )
@@
     (stroke (width 0) (type default))
   )
+  (wire (pts (xy 172.72 71.12) (xy 172.72 76.2))
+    (stroke (width 0) (type default))
+  )
   (wire (pts (xy 139.7 69.85) (xy 139.7 59.69))
     (stroke (width 0) (type default))
@@
     (stroke (width 0) (type default))
   )
-  (wire (pts (xy 143.51 74.93) (xy 172.72 74.93))
+  (wire (pts (xy 143.51 76.2) (xy 172.72 76.2))
     (stroke (width 0) (type default))
   )
@@
     (stroke (width 0) (type default))
   )
-  (wire (pts (xy 172.72 74.93) (xy 172.72 71.12))
-    (stroke (width 0) (type default))
-  )
-  (wire (pts (xy 143.51 74.93) (xy 143.51 64.77))
+  (wire (pts (xy 143.51 76.2) (xy 143.51 64.77))
     (stroke (width 0) (type default))
   )
@@
     (effects (font (size 1.27 1.27)) (justify left bottom))
   )
-  (global_label "module -VCC" (shape input) (at 148.59 71.12 0) (fields_autoplaced)
+  (global_label "module -VCC" (shape input) (at 148.59 72.39 0) (fields_autoplaced)
     (effects (font (size 1.27 1.27)) (justify left))
-    (property "Intersheetrefs" "${INTERSHEET_REFS}" (at 166.815 71.12 0)
+    (property "Intersheetrefs" "${INTERSHEET_REFS}" (at 166.815 72.39 0)
       (effects (font (size 1.27 1.27)) (justify left) hide)
     )
@@
         (path "/1ce81232-195d-4047-8575-458c62622b55"
           (reference "#PWR?") (unit 1)
-        )
-      )
-    )
-  )
-  (symbol (lib_id "power:PWR_FLAG") (at 148.59 69.85 90) (unit 1)
-    (in_bom yes) (on_board yes) (dnp no) (fields_autoplaced)
-    (property "Reference" "#FLG02" (at 146.685 69.85 0)
-      (effects (font (size 1.27 1.27)) hide)
-    )
-    (property "Value" "PWR_FLAG" (at 143.51 69.85 0)
-      (effects (font (size 1.27 1.27)) hide)
-    )
-    (property "Footprint" "" (at 148.59 69.85 0)
-      (effects (font (size 1.27 1.27)) hide)
-    )
-    (property "Datasheet" "~" (at 148.59 69.85 0)
-      (effects (font (size 1.27 1.27)) hide)
-    )
-    (pin "1")
-    (instances
-      (project "lowPassSecondOrderSK"
-        (path "/1abb811e-e6a2-481c-ab83-294d796176de"
-          (reference "#FLG02") (unit 1)
-        )
-      )
-      (project "kicad"
-        (path "/1ce81232-195d-4047-8575-458c62622b55"
-          (reference "#FLG?") (unit 1)
         )
       )
@@
     )
   )
-  (symbol (lib_id "power:PWR_FLAG") (at 148.59 54.61 90) (unit 1)
-    (in_bom yes) (on_board yes) (dnp no) (fields_autoplaced)
-    (property "Reference" "#FLG01" (at 146.685 54.61 0)
-      (effects (font (size 1.27 1.27)) hide)
-    )
-    (property "Value" "PWR_FLAG" (at 143.51 54.61 0)
-      (effects (font (size 1.27 1.27)) hide)
-    )
-    (property "Footprint" "" (at 148.59 54.61 0)
-      (effects (font (size 1.27 1.27)) hide)
-    )
-    (property "Datasheet" "~" (at 148.59 54.61 0)
-      (effects (font (size 1.27 1.27)) hide)
-    )
-    (pin "1")
-    (instances
-      (project "lowPassSecondOrderSK"
-        (path "/1abb811e-e6a2-481c-ab83-294d796176de"
-          (reference "#FLG01") (unit 1)
-        )
-      )
-      (project "kicad"
-        (path "/1ce81232-195d-4047-8575-458c62622b55"
-          (reference "#FLG?") (unit 1)
-        )
-      )
-    )
-  )
-  (symbol (lib_id "Device:R") (at 172.72 78.74 0) (mirror x) (unit 1)
-    (in_bom yes) (on_board yes) (dnp no)
-    (property "Reference" "R4" (at 176.53 80.01 90)
+  (symbol (lib_id "Device:R") (at 172.72 80.01 0) (mirror x) (unit 1)
+    (in_bom yes) (on_board yes) (dnp no)
+    (property "Reference" "R4" (at 175.26 78.74 90)
       (effects (font (size 1.27 1.27)) (justify left))
     )
-    (property "Value" "R" (at 176.53 77.47 90)
-      (effects (font (size 1.27 1.27)) (justify left) hide)
-    )
-    (property "Footprint" "Resistor_THT:R_Axial_DIN0207_L6.3mm_D2.5mm_P7.62mm_Horizontal" (at 170.942 78.74 90)
-      (effects (font (size 1.27 1.27)) hide)
-    )
-    (property "Datasheet" "~" (at 172.72 78.74 0)
+    (property "Value" "R" (at 176.53 78.74 90)
+      (effects (font (size 1.27 1.27)) (justify left) hide)
+    )
+    (property "Footprint" "Resistor_THT:R_Axial_DIN0207_L6.3mm_D2.5mm_P7.62mm_Horizontal" (at 170.942 80.01 90)
+      (effects (font (size 1.27 1.27)) hide)
+    )
+    (property "Datasheet" "~" (at 172.72 80.01 0)
       (effects (font (size 1.27 1.27)) hide)
     )
@@
   (symbol (lib_id "Device:R") (at 172.72 67.31 0) (unit 1)
     (in_bom yes) (on_board yes) (dnp no)
-    (property "Reference" "R3" (at 175.26 66.04 0)
+    (property "Reference" "R3" (at 175.26 68.58 90)
       (effects (font (size 1.27 1.27)) (justify left))
     )
@@
     )
   )
-  (symbol (lib_id "power:GND") (at 172.72 82.55 0) (unit 1)
-    (in_bom yes) (on_board yes) (dnp no)
-    (property "Reference" "#PWR02" (at 172.72 88.9 0)
-      (effects (font (size 1.27 1.27)) hide)
-    )
-    (property "Value" "GND" (at 172.72 86.36 0)
-      (effects (font (size 1.27 1.27)) hide)
-    )
-    (property "Footprint" "" (at 172.72 82.55 0)
-      (effects (font (size 1.27 1.27)) hide)
-    )
-    (property "Datasheet" "" (at 172.72 82.55 0)
-      (effects (font (size 1.27 1.27)) hide)
-    )
+  (symbol (lib_id "power:GND") (at 172.72 83.82 0) (unit 1)
+    (in_bom yes) (on_board yes) (dnp no)
+    (property "Reference" "#PWR02" (at 172.72 90.17 0)
+      (effects (font (size 1.27 1.27)) hide)
+    )
+    (property "Value" "GND" (at 172.72 87.63 0)
+      (effects (font (size 1.27 1.27)) hide)
+    )
+    (property "Footprint" "" (at 172.72 83.82 0)
+      (effects (font (size 1.27 1.27)) hide)
+    )
+    (property "Datasheet" "" (at 172.72 83.82 0)
+      (effects (font (size 1.27 1.27)) hide)
+    )
