File: modules/nonInversor/nonInversor.kicad_sch (KiCad schematic)
At the start: 4 parts

Commit message: Little changes on each schematic
Changed lines of the file:
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@@
+    (stroke (width 0) (type default))
+  )
+  (wire (pts (xy 158.75 113.03) (xy 158.75 110.49))
     (stroke (width 0) (type default))
   )
@@
     )
   )
-  (global_label "module -VCC" (shape input) (at 158.75 110.49 0) (fields_autoplaced)
+  (global_label "module -VCC" (shape input) (at 158.75 113.03 0) (fields_autoplaced)
     (effects (font (size 1.27 1.27)) (justify left))
-    (property "Intersheetrefs" "${INTERSHEET_REFS}" (at 178.1845 110.49 0)
+    (property "Intersheetrefs" "${INTERSHEET_REFS}" (at 178.1845 113.03 0)
       (effects (font (size 1.27 1.27)) (justify left) hide)
     )
@@
         (path "/49a8d326-328c-4424-88b7-483ea059f0a8"
           (reference "#PWR02") (unit 1)
-        )
-      )
-    )
-  )
-  (symbol (lib_id "power:PWR_FLAG") (at 158.75 110.49 90) (unit 1)
-    (in_bom yes) (on_board yes) (dnp no) (fields_autoplaced)
-    (property "Reference" "#FLG?" (at 156.845 110.49 0)
-      (effects (font (size 1.27 1.27)) hide)
-    )
-    (property "Value" "PWR_FLAG" (at 153.67 110.49 0)
-      (effects (font (size 1.27 1.27)) hide)
-    )
-    (property "Footprint" "" (at 158.75 110.49 0)
-      (effects (font (size 1.27 1.27)) hide)
-    )
-    (property "Datasheet" "~" (at 158.75 110.49 0)
-      (effects (font (size 1.27 1.27)) hide)
-    )
-    (pin "1")
-    (instances
-      (project "kicad"
-        (path "/1ce81232-195d-4047-8575-458c62622b55"
-          (reference "#FLG?") (unit 1)
-        )
-      )
-      (project "nonInversor"
-        (path "/49a8d326-328c-4424-88b7-483ea059f0a8"
-          (reference "#FLG02") (unit 1)
         )
       )
@@
         )
       )
-    )
-  )
-  (symbol (lib_id "power:PWR_FLAG") (at 158.75 95.25 90) (unit 1)
-    (in_bom yes) (on_board yes) (dnp no) (fields_autoplaced)
-    (property "Reference" "#FLG?" (at 156.845 95.25 0)
-      (effects (font (size 1.27 1.27)) hide)
-    )
-    (property "Value" "PWR_FLAG" (at 153.67 95.25 0)
-      (effects (font (size 1.27 1.27)) hide)
-    )
-    (property "Footprint" "" (at 158.75 95.25 0)
-      (effects (font (size 1.27 1.27)) hide)
-    )
-    (property "Datasheet" "~" (at 158.75 95.25 0)
-      (effects (font (size 1.27 1.27)) hide)
-    )
-    (pin "1")
-    (instances
-      (project "kicad"
-        (path "/1ce81232-195d-4047-8575-458c62622b55"
-          (reference "#FLG?") (unit 1)
-        )
-      )
-      (project "nonInversor"
-        (path "/49a8d326-328c-4424-88b7-483ea059f0a8"
-          (reference "#FLG01") (unit 1)
-        )
-      )
