File: modules/notchSecondOrderTwint/notchSecondOrderTwint.kicad_sch (KiCad schematic)
At the start: 10 parts

Commit message: Update moudules
Parts:
- removed R?: R, Resistor_THT:R_Axial_DIN0207_L6.3mm_D2.5mm_P7.62mm_Horizontal, symbol Device:R
- added R?: R, Resistor_THT:R_Axial_DIN0207_L6.3mm_D2.5mm_P7.62mm_Horizontal, symbol Device:R
Connections:
- net GND: now also R?.1
- net at R?.2: now also U?.2 (-), R?.2
Changed lines of the file:
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@@
   (junction (at 147.32 102.87) (diameter 0) (color 0 0 0 0)
+  )
+  (junction (at 147.32 115.57) (diameter 0) (color 0 0 0 0)
   )
   (junction (at 111.76 110.49) (diameter 0) (color 0 0 0 0)
@@
     (stroke (width 0) (type default))
   )
-  (wire (pts (xy 139.7 115.57) (xy 147.32 115.57))
-    (stroke (width 0) (type default))
-  )
   (wire (pts (xy 147.32 115.57) (xy 147.32 111.76))
     (stroke (width 0) (type default))
@@
     (stroke (width 0) (type default))
   )
-  (wire (pts (xy 132.08 115.57) (xy 118.11 115.57))
+  (wire (pts (xy 118.11 115.57) (xy 147.32 115.57))
     (stroke (width 0) (type default))
   )
@@
     )
   )
+  (symbol (lib_id "Device:R") (at 147.32 119.38 0) (mirror x) (unit 1)
+    (in_bom yes) (on_board yes) (dnp no)
+    (property "Reference" "R?" (at 151.13 120.65 90)
+      (effects (font (size 1.27 1.27)) (justify left))
+    )
+    (property "Value" "R" (at 151.13 118.11 90)
+      (effects (font (size 1.27 1.27)) (justify left) hide)
+    )
+    (property "Footprint" "Resistor_THT:R_Axial_DIN0207_L6.3mm_D2.5mm_P7.62mm_Horizontal" (at 145.542 119.38 90)
+      (effects (font (size 1.27 1.27)) hide)
+    )
+    (property "Datasheet" "~" (at 147.32 119.38 0)
+      (effects (font (size 1.27 1.27)) hide)
+    )
+    (pin "1")
+    (pin "2")
+    (instances
+      (project "kicad"
+        (path "/1ce81232-195d-4047-8575-458c62622b55"
+          (reference "R?") (unit 1)
+        )
+      )
+      (project "notchSecondOrderTwint"
+        (path "/333366c1-a3d2-4393-8688-1e46c1ff01f1"
+          (reference "R4") (unit 1)
+        )
+      )
+    )
+  )
   (symbol (lib_id "power:PWR_FLAG") (at 123.19 110.49 90) (unit 1)
     (in_bom yes) (on_board yes) (dnp no) (fields_autoplaced)
@@
         (path "/333366c1-a3d2-4393-8688-1e46c1ff01f1"
           (reference "#FLG02") (unit 1)
+        )
+      )
+    )
+  )
+  (symbol (lib_id "power:GND") (at 147.32 123.19 0) (unit 1)
+    (in_bom yes) (on_board yes) (dnp no)
+    (property "Reference" "#PWR?" (at 147.32 129.54 0)
+      (effects (font (size 1.27 1.27)) hide)
+    )
+    (property "Value" "GND" (at 147.32 127 0)
+      (effects (font (size 1.27 1.27)) hide)
+    )
+    (property "Footprint" "" (at 147.32 123.19 0)
+      (effects (font (size 1.27 1.27)) hide)
+    )
+    (property "Datasheet" "" (at 147.32 123.19 0)
+      (effects (font (size 1.27 1.27)) hide)
+    )
+    (pin "1")
+    (instances
+      (project "kicad"
+        (path "/1ce81232-195d-4047-8575-458c62622b55"
+          (reference "#PWR?") (unit 1)
+        )
+      )
+      (project "notchSecondOrderTwint"
+        (path "/333366c1-a3d2-4393-8688-1e46c1ff01f1"
+          (reference "#PWR03") (unit 1)
         )
       )
@@
         )
       )
-    )
-  )
-  (symbol (lib_id "Device:R") (at 135.89 115.57 90) (mirror x) (unit 1)
-    (in_bom yes) (on_board yes) (dnp no)
-    (property "Reference" "R?" (at 134.62 119.38 90)
-      (effects (font (size 1.27 1.27)) (justify left))
-    )
-    (property "Value" "R" (at 137.16 119.38 90)
-      (effects (font (size 1.27 1.27)) (justify left) hide)
-    )
-    (property "Footprint" "Resistor_THT:R_Axial_DIN0207_L6.3mm_D2.5mm_P7.62mm_Horizontal" (at 135.89 113.792 90)
-      (effects (font (size 1.27 1.27)) hide)
-    )
-    (property "Datasheet" "~" (at 135.89 115.57 0)
-      (effects (font (size 1.27 1.27)) hide)
-    )
-    (pin "1")
-    (pin "2")
-    (instances
-      (project "kicad"
-        (path "/1ce81232-195d-4047-8575-458c62622b55"
-          (reference "R?") (unit 1)
-        )
-      )
-      (project "notchSecondOrderTwint"
-        (path "/333366c1-a3d2-4393-8688-1e46c1ff01f1"
-          (reference "R4") (unit 1)
-        )
-      )

Commit message: Little changes on each schematic
Other:
- moved on the sheet: R?
Changed lines of the file:
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@@
   (junction (at 102.87 101.6) (diameter 0) (color 0 0 0 0)
   )
-  (junction (at 123.19 110.49) (diameter 0) (color 0 0 0 0)
+  (junction (at 147.32 116.84) (diameter 0) (color 0 0 0 0)
   )
   (junction (at 102.87 99.06) (diameter 0) (color 0 0 0 0)
@@
   )
   (junction (at 147.32 102.87) (diameter 0) (color 0 0 0 0)
-  )
-  (junction (at 147.32 115.57) (diameter 0) (color 0 0 0 0)
   )
   (junction (at 111.76 110.49) (diameter 0) (color 0 0 0 0)
@@
     (stroke (width 0) (type default))
   )
-  (wire (pts (xy 147.32 115.57) (xy 147.32 111.76))
-    (stroke (width 0) (type default))
-  )
   (wire (pts (xy 114.3 100.33) (xy 114.3 110.49))
     (stroke (width 0) (type default))
@@
     (stroke (width 0) (type default))
   )
-  (wire (pts (xy 123.19 111.76) (xy 123.19 110.49))
+  (wire (pts (xy 123.19 113.03) (xy 123.19 110.49))
     (stroke (width 0) (type default))
   )
@@
     (stroke (width 0) (type default))
   )
-  (wire (pts (xy 118.11 115.57) (xy 147.32 115.57))
+  (wire (pts (xy 118.11 118.11) (xy 147.32 118.11))
     (stroke (width 0) (type default))
   )
@@
     (stroke (width 0) (type default))
   )
+  (wire (pts (xy 147.32 118.11) (xy 147.32 116.84))
+    (stroke (width 0) (type default))
+  )
   (wire (pts (xy 102.87 99.06) (xy 102.87 101.6))
     (stroke (width 0) (type default))
@@
     (stroke (width 0) (type default))
   )
-  (wire (pts (xy 118.11 115.57) (xy 118.11 105.41))
+  (wire (pts (xy 118.11 118.11) (xy 118.11 105.41))
     (stroke (width 0) (type default))
   )
   (wire (pts (xy 91.44 101.6) (xy 102.87 101.6))
+    (stroke (width 0) (type default))
+  )
+  (wire (pts (xy 147.32 111.76) (xy 147.32 116.84))
     (stroke (width 0) (type default))
   )
@@
     (fill (type none))
   )
-  (text "Circuito Notch Twint 2ª Ordem" (at 137.16 128.27 0)
+  (text "Circuito Notch Twint 2ª Ordem" (at 142.24 129.54 0)
     (effects (font (size 1.27 1.27)) (justify left bottom))
   )
@@
     )
   )
-  (global_label "module -VCC" (shape input) (at 123.19 111.76 0) (fields_autoplaced)
+  (global_label "module -VCC" (shape input) (at 123.19 113.03 0) (fields_autoplaced)
     (effects (font (size 1.27 1.27)) (justify left))
-    (property "Intersheetrefs" "${INTERSHEET_REFS}" (at 142.6245 111.76 0)
+    (property "Intersheetrefs" "${INTERSHEET_REFS}" (at 142.6245 113.03 0)
       (effects (font (size 1.27 1.27)) (justify left) hide)
     )
@@
   (symbol (lib_id "Device:R") (at 147.32 107.95 0) (unit 1)
     (in_bom yes) (on_board yes) (dnp no)
-    (property "Reference" "R?" (at 149.86 106.68 0)
+    (property "Reference" "R?" (at 149.86 109.22 90)
       (effects (font (size 1.27 1.27)) (justify left))
     )
@@
   (symbol (lib_id "Device:C") (at 99.06 110.49 90) (unit 1)
     (in_bom yes) (on_board yes) (dnp no)
-    (property "Reference" "C?" (at 97.79 114.3 90)
+    (property "Reference" "C?" (at 99.06 114.3 90)
       (effects (font (size 1.27 1.27)))
     )
@@
   (symbol (lib_id "Device:C") (at 114.3 114.3 180) (unit 1)
     (in_bom yes) (on_board yes) (dnp no)
-    (property "Reference" "C?" (at 118.11 115.57 90)
+    (property "Reference" "C?" (at 118.11 114.3 90)
       (effects (font (size 1.27 1.27)))
     )
@@
     )
   )
-  (symbol (lib_id "Device:R") (at 147.32 119.38 0) (mirror x) (unit 1)
-    (in_bom yes) (on_board yes) (dnp no)
-    (property "Reference" "R?" (at 151.13 120.65 90)
+  (symbol (lib_id "Device:R") (at 147.32 120.65 0) (mirror x) (unit 1)
+    (in_bom yes) (on_board yes) (dnp no)
+    (property "Reference" "R?" (at 149.86 119.38 90)
       (effects (font (size 1.27 1.27)) (justify left))
     )
-    (property "Value" "R" (at 151.13 118.11 90)
-      (effects (font (size 1.27 1.27)) (justify left) hide)
-    )
-    (property "Footprint" "Resistor_THT:R_Axial_DIN0207_L6.3mm_D2.5mm_P7.62mm_Horizontal" (at 145.542 119.38 90)
-      (effects (font (size 1.27 1.27)) hide)
-    )
-    (property "Datasheet" "~" (at 147.32 119.38 0)
+    (property "Value" "R" (at 151.13 119.38 90)
+      (effects (font (size 1.27 1.27)) (justify left) hide)
+    )
+    (property "Footprint" "Resistor_THT:R_Axial_DIN0207_L6.3mm_D2.5mm_P7.62mm_Horizontal" (at 145.542 120.65 90)
+      (effects (font (size 1.27 1.27)) hide)
+    )
+    (property "Datasheet" "~" (at 147.32 120.65 0)
       (effects (font (size 1.27 1.27)) hide)
     )
@@
     )
   )
-  (symbol (lib_id "power:PWR_FLAG") (at 123.19 110.49 90) (unit 1)
-    (in_bom yes) (on_board yes) (dnp no) (fields_autoplaced)
-    (property "Reference" "#FLG?" (at 121.285 110.49 0)
-      (effects (font (size 1.27 1.27)) hide)
-    )
-    (property "Value" "PWR_FLAG" (at 118.11 110.49 0)
-      (effects (font (size 1.27 1.27)) hide)
-    )
-    (property "Footprint" "" (at 123.19 110.49 0)
-      (effects (font (size 1.27 1.27)) hide)
-    )
-    (property "Datasheet" "~" (at 123.19 110.49 0)
-      (effects (font (size 1.27 1.27)) hide)
-    )
-    (pin "1")
-    (instances
-      (project "kicad"
-        (path "/1ce81232-195d-4047-8575-458c62622b55"
-          (reference "#FLG?") (unit 1)
-        )
-      )
-      (project "notchSecondOrderTwint"
-        (path "/333366c1-a3d2-4393-8688-1e46c1ff01f1"
-          (reference "#FLG02") (unit 1)
-        )
-      )
-    )
-  )
-  (symbol (lib_id "power:GND") (at 147.32 123.19 0) (unit 1)
-    (in_bom yes) (on_board yes) (dnp no)
-    (property "Reference" "#PWR?" (at 147.32 129.54 0)
-      (effects (font (size 1.27 1.27)) hide)
-    )
-    (property "Value" "GND" (at 147.32 127 0)
-      (effects (font (size 1.27 1.27)) hide)
-    )
-    (property "Footprint" "" (at 147.32 123.19 0)
-      (effects (font (size 1.27 1.27)) hide)
-    )
-    (property "Datasheet" "" (at 147.32 123.19 0)
+  (symbol (lib_id "power:GND") (at 147.32 124.46 0) (unit 1)
+    (in_bom yes) (on_board yes) (dnp no)
+    (property "Reference" "#PWR?" (at 147.32 130.81 0)
+      (effects (font (size 1.27 1.27)) hide)
+    )
+    (property "Value" "GND" (at 147.32 128.27 0)
+      (effects (font (size 1.27 1.27)) hide)
+    )
+    (property "Footprint" "" (at 147.32 124.46 0)
+      (effects (font (size 1.27 1.27)) hide)
+    )
+    (property "Datasheet" "" (at 147.32 124.46 0)
       (effects (font (size 1.27 1.27)) hide)
     )
@@
     )
   )
-  (symbol (lib_id "power:PWR_FLAG") (at 123.19 95.25 90) (unit 1)
-    (in_bom yes) (on_board yes) (dnp no) (fields_autoplaced)
-    (property "Reference" "#FLG?" (at 121.285 95.25 0)
-      (effects (font (size 1.27 1.27)) hide)
-    )
-    (property "Value" "PWR_FLAG" (at 118.11 95.25 0)
-      (effects (font (size 1.27 1.27)) hide)
-    )
-    (property "Footprint" "" (at 123.19 95.25 0)
-      (effects (font (size 1.27 1.27)) hide)
-    )
-    (property "Datasheet" "~" (at 123.19 95.25 0)
-      (effects (font (size 1.27 1.27)) hide)
-    )
-    (pin "1")
-    (instances
-      (project "kicad"
-        (path "/1ce81232-195d-4047-8575-458c62622b55"
-          (reference "#FLG?") (unit 1)
-        )
-      )
-      (project "notchSecondOrderTwint"
-        (path "/333366c1-a3d2-4393-8688-1e46c1ff01f1"
-          (reference "#FLG01") (unit 1)
-        )
-      )
-    )
-  )
   (symbol (lib_id "Device:C") (at 104.14 118.11 270) (unit 1)
     (in_bom yes) (on_board yes) (dnp no)
-    (property "Reference" "C?" (at 106.68 114.3 90)
+    (property "Reference" "C?" (at 104.14 121.92 90)
       (effects (font (size 1.27 1.27)))
     )
